File: 201904_Esp32ReprapController.sch (KiCad schematic (older format))
At the start: 60 parts, among them J1 24V_IN, J10 NOZZLE, J11 BED, J110 MOTOR_X, J12 FAN1, J120 MOTOR_Y, J13 FAN2, J130 MOTOR_Z, J14 FAN_ALWAYS, J140 MOTOR_E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

Commit message: board r2 (never built)
Parts:
- removed Q3: IRLZ44N, Felix_Common:TO-220-3_Vertical_LongPads, symbol Device:Q_NMOS_GDS
- removed R14: 10, Felix_Common:R_Axial_DIN0207_L6.3mm_D2.5mm_P10.16mm_Horizontal, symbol Device:R
- removed R15: 100k, Felix_Common:R_Axial_DIN0207_L6.3mm_D2.5mm_P10.16mm_Horizontal, symbol Device:R
- removed R160: 4.7k, Felix_Common:R_Axial_DIN0207_L6.3mm_D2.5mm_P10.16mm_Horizontal, symbol Device:R
- removed R161: R, Felix_Common:R_Axial_DIN0207_L6.3mm_D2.5mm_P10.16mm_Horizontal, symbol Device:R
- added C1, C3: 100uF, Felix_Common:CP_Radial_D6.3mm_P2.50mm, symbol Device:CP
- added C2, C21, C23, C4: 0.1uF, Felix_Common:C_Rect_L7.2mm_W2.5mm_P5.00mm_FKS2_FKP2_MKS2_MKP2, symbol Device:C
- added U5: ULN2803A, Felix_Common:DIP-18_W7.62mm_Socket_LongPads, symbol Transistor_Array:ULN2803A
- C20: symbol Device:C -> Device:CP
- C22: renamed from C21; symbol Device:C -> Device:CP
- J14: value FAN_ALWAYS -> FAN3
- renumbered R21 to R22
Connections:
- net +24V: now also U5.10 (COM)
- net +5V: now also C1.1, C2.1
- net BED_T: now also C21.1
- net GND: now also C1.2, C2.2, C21.2, C23.2, C3.2, C4.2, U5.9 (GND); no longer J14.2 (Pin_2)
- net I2S_BCK: now also U1.9 (IO25); no longer U1.10 (IO26)
- net I2S_WS: now also U1.10 (IO26); no longer U1.9 (IO25)
- net NOZZLE_T: now also C23.1
- net Q140: now also U5.4 (I4), U5.5 (I5), U5.6 (I6)
- net Q141: now also U5.7 (I7), U5.8 (I8)
- net VCC: now also C3.1, C4.1
- net at J12.2 (Pin_2): now also U5.16 (O3), U5.17 (O2), U5.18 (O1); no longer J13.2 (Pin_2)
- net FAN renamed FAN1
- net FAN1: now also U5.1 (I1), U5.2 (I2), U5.3 (I3)
- new net: J14.2 (Pin_2), U5.11 (O8), U5.12 (O7)
- new net: J13.2 (Pin_2), U5.13 (O6), U5.14 (O5), U5.15 (O4)
- no-connect marks 31 -> 29
Other:
- moved on the sheet: J12, J13, J14, J20, J21, R22

Commit message: board r3 (milled and built 2019-06)
Parts:
- added D2: LED_NOZ, Felix_Common:LED_D5.0mm, symbol Device:LED
- added D3: LED_BED, Felix_Common:LED_D5.0mm, symbol Device:LED
- added R12, R17: 2.2k, Felix_Common:R_Axial_DIN0207_L6.3mm_D2.5mm_P10.16mm_Horizontal, symbol Device:R
- renumbered R12 to R15, R13 to R16
Connections:
- net Q142 is gone; now on net Q142_FAN2: U4.6 (QG)
- net Q143 is gone; now on net Q143_FAN3: U4.7 (QH)
- net +24V: now also D2.2 (A), D3.2 (A)
- net BEEPER: no longer U1.31 (IO16)
- net Q128: no longer A1.15 (STEP)
- net Q136: no longer A3.9 (~ENABLE)
- net ~RESET: no longer U1.2 (EN)
- net at J10.2 (Pin_2), Q1.2 (D): now also R12.2
- net at J11.2 (Pin_2), Q2.2 (D): now also R17.2
- net BED renamed IO4_BED
- net BED_T renamed I36_T_BED
- net I36_T_BED: now also U1.3 (SVP-I36); no longer U1.4 (SVN-I39)
- net BTN_EN1 renamed IO12_LCD_EN
- net IO12_LCD_EN: now also J40.8 (Pin_8); no longer J40.3 (Pin_3)
- net BTN_EN2 renamed IO14_LCD_D4
- net IO14_LCD_D4: now also J40.6 (Pin_6); no longer J40.5 (Pin_5)
- net BTN_ENC renamed IO27_BTN_ENC
- net IO27_BTN_ENC: now also U1.11 (IO27); no longer U1.8 (IO33)
- net FAN1 renamed IO13_FAN1
- net I2S_BCK renamed IO22_I2S_BCK
- net IO22_I2S_BCK: now also U1.22 (IO22); no longer U1.9 (IO25)
- net I2S_DATA renamed IO21_I2S_DATA
- net IO21_I2S_DATA: now also U1.25 (IO21); no longer U1.11 (IO27)
- net I2S_WS renamed IO17_I2S_WS
- net IO17_I2S_WS: now also U1.30 (IO17); no longer U1.10 (IO26)
- removed net LCD_D4: J40.6 (Pin_6), U1.22 (IO22)
- removed net LCD_EN: J40.8 (Pin_8), U1.25 (IO21)
- net LCD_RS renamed IO33_LCD_RS
- net IO33_LCD_RS: now also U1.8 (IO33); no longer U1.30 (IO17)
- net NOZZLE renamed IO2_NOZZLE
- net NOZZLE_T renamed I39_T_NOZ
- net I39_T_NOZ: now also U1.4 (SVN-I39); no longer U1.3 (SVP-I36)
- net Q129 renamed Q129_Z_DIR
- net Q129_Z_DIR: now also A3.16 (DIR); no longer A1.16 (DIR)
- net Q130 renamed Q130_Z_STEP
- net Q130_Z_STEP: now also A3.15 (STEP); no longer A1.9 (~ENABLE)
- net Q131 renamed Q131_Z_EN
- net Q131_Z_EN: now also A3.9 (~ENABLE); no longer A2.15 (STEP)
- net Q132 renamed Q132_Y_DIR
- net Q133 renamed Q133_Y_STEP
- net Q133_Y_STEP: now also A2.15 (STEP); no longer A2.9 (~ENABLE)
- net Q134 renamed Q134_Y_EN
- net Q134_Y_EN: now also A2.9 (~ENABLE); no longer A3.15 (STEP)
- net Q135 renamed Q135_X_DIR
- net Q135_X_DIR: now also A1.16 (DIR); no longer A3.16 (DIR)
- net Q137 renamed Q137_X_STEP
- net Q137_X_STEP: now also A1.15 (STEP); no longer A4.15 (STEP)
- net Q138 renamed Q138_X_EN
- net Q138_X_EN: now also A1.9 (~ENABLE); no longer A4.16 (DIR)
- net Q139 renamed Q139_E_EN
- net Q140 renamed Q142_FAN2
- net Q142_FAN2: no longer U4.4 (QE)
- net Q141 renamed Q143_FAN3
- net Q143_FAN3: no longer U4.5 (QF)
- net SERVO renamed IO15_SERVO
- net IO15_SERVO: now also U1.35 (IO15); no longer U1.7 (IO32)
- net X_MIN renamed IO34_X_MIN
- net Y_MIN renamed IO35_Y_MIN
- net Z_MIN renamed IO32_Z_MIN
- net IO32_Z_MIN: now also U1.7 (IO32); no longer U1.35 (IO15)
- new net: D2.1 (K), R12.1
- new net: D3.1 (K), R17.1
- new net IO25_BTN_EN2: J40.5 (Pin_5), U1.9 (IO25)
- new net IO26_BTN_EN1: J40.3 (Pin_3), U1.10 (IO26)
- new net Q140_E_STEP: A4.15 (STEP), U4.4 (QE)
- new net Q141_E_DIR: A4.16 (DIR), U4.5 (QF)
- new net ~ESP32_EN: U1.2 (EN)
- no-connect marks 29 -> 33
Other:
- moved on the sheet: C30, C31, C32, J10, J11, J30, J31, J32, Q2, R15, R16, R30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

Commit message: cosmetics
Parts:
- D2: value LED_NOZ -> NOZ
- D3: value LED_BED -> BED
- F1: value 3A (Rest) -> 3A REM
- F2: value 10A (Bed) -> 10A BED
- J1: value 24V_IN -> -24V IN+
- J10: value NOZZLE -> +NOZ-
- J11: value BED -> +BED-
- J110: value MOTOR_X -> MOT X
- J12: value FAN1 -> +FAN1-
- J120: value MOTOR_Y -> MOT Y
- J13: value FAN2 -> +FAN2-
- J130: value MOTOR_Z -> MOT Z
- J14: value FAN3 -> +FAN3-
- J140: value MOTOR_E -> MOT E
- J20: value BED_T -> +BT-
- J21: value NOZZLE_T -> +NT-
- J30: value Conn_X_Min -> +XM-
- J31: value Conn_Y_Min -> +YM-
- J32: value Conn_Z_Min -> +ZM-
- J50: value SD_Card -> SD GND
Changed lines of the file:
@@
 P 15000 1850
 F 0 "J110" H 14950 2050 50  0000 L CNN
-F 1 "MOTOR_X" V 15100 1550 50  0000 L CNN
+F 1 "MOT X" V 15100 1800 50  0000 C CNN
 F 2 "Felix_Common:PinHeader_1x04_P2.54mm_Vertical_LongPads" H 15000 1850 50  0001 C CNN
 F 3 "~" H 15000 1850 50  0001 C CNN
@@
 P 5500 6050
 F 0 "J30" H 5580 6092 50  0000 L CNN
-F 1 "Conn_X_Min" H 5580 6001 50  0000 L CNN
+F 1 "+XM-" H 5580 6001 50  0000 L CNN
 F 2 "Felix_Common:PinHeader_1x02_P2.54mm_Vertical_LongPads" H 5500 6050 50  0001 C CNN
 F 3 "~" H 5500 6050 50  0001 C CNN
@@
 P 6600 6050
 F 0 "J31" H 6680 6092 50  0000 L CNN
-F 1 "Conn_Y_Min" H 6680 6001 50  0000 L CNN
+F 1 "+YM-" H 6680 6001 50  0000 L CNN
 F 2 "Felix_Common:PinHeader_1x02_P2.54mm_Vertical_LongPads" H 6600 6050 50  0001 C CNN
 F 3 "~" H 6600 6050 50  0001 C CNN
@@
 P 7700 6050
 F 0 "J32" H 7780 6092 50  0000 L CNN
-F 1 "Conn_Z_Min" H 7780 6001 50  0000 L CNN
+F 1 "+ZM-" H 7780 6001 50  0000 L CNN
 F 2 "Felix_Common:PinHeader_1x02_P2.54mm_Vertical_LongPads" H 7700 6050 50  0001 C CNN
 F 3 "~" H 7700 6050 50  0001 C CNN
@@
 P 15000 4250
 F 0 "J120" H 14950 4450 50  0000 L CNN
-F 1 "MOTOR_Y" V 15100 3950 50  0000 L CNN
+F 1 "MOT Y" V 15100 4200 50  0000 C CNN
 F 2 "Felix_Common:PinHeader_1x04_P2.54mm_Vertical_LongPads" H 15000 4250 50  0001 C CNN
 F 3 "~" H 15000 4250 50  0001 C CNN
@@
 P 15000 6650
 F 0 "J130" H 14950 6850 50  0000 L CNN
-F 1 "MOTOR_Z" V 15100 6350 50  0000 L CNN
+F 1 "MOT Z" V 15100 6600 50  0000 C CNN
 F 2 "Felix_Common:PinHeader_1x04_P2.54mm_Vertical_LongPads" H 15000 6650 50  0001 C CNN
 F 3 "~" H 15000 6650 50  0001 C CNN
@@
 P 12800 6650
 F 0 "J140" H 12750 6850 50  0000 L CNN
-F 1 "MOTOR_E" V 12900 6350 50  0000 L CNN
+F 1 "MOT E" V 12900 6600 50  0000 C CNN
 F 2 "Felix_Common:PinHeader_1x04_P2.54mm_Vertical_LongPads" H 12800 6650 50  0001 C CNN
 F 3 "~" H 12800 6650 50  0001 C CNN
@@
 P 1050 2150
 F 0 "J1" H 970 1825 50  0000 C CNN
-F 1 "24V_IN" H 970 1916 50  0000 C CNN
+F 1 "-24V IN+" H 970 1916 50  0000 C CNN
 F 2 "Felix_Common:TerminalBlock_ScrewTerminal_1x02_P5.00mm_Horizontal" H 1050 2150 50  0001 C CNN
 F 3 "~" H 1050 2150 50  0001 C CNN
@@
 P 2550 5200
 F 0 "J11" H 2630 5192 50  0000 L CNN
-F 1 "BED" H 2630 5101 50  0000 L CNN
+F 1 "+BED-" H 2630 5101 50  0000 L CNN
 F 2 "Felix_Common:TerminalBlock_ScrewTerminal_1x02_P5.00mm_Horizontal" H 2550 5200 50  0001 C CNN
 F 3 "~" H 2550 5200 50  0001 C CNN
@@
 P 2550 3950
 F 0 "J10" H 2629 3942 50  0000 L CNN
-F 1 "NOZZLE" H 2629 3851 50  0000 L CNN
+F 1 "+NOZ-" H 2629 3851 50  0000 L CNN
 F 2 "Felix_Common:TerminalBlock_ScrewTerminal_1x02_P5.00mm_Horizontal" H 2550 3950 50  0001 C CNN
 F 3 "~" H 2550 3950 50  0001 C CNN
@@
 P 2750 7050
 F 0 "J14" H 2829 7042 50  0000 L CNN
-F 1 "FAN3" H 2829 6951 50  0000 L CNN
+F 1 "+FAN3-" H 2829 6951 50  0000 L CNN
 F 2 "Felix_Common:TerminalBlock_ScrewTerminal_1x02_P5.00mm_Horizontal" H 2750 7050 50  0001 C CNN
 F 3 "~" H 2750 7050 50  0001 C CNN
@@
 P 2750 6350
 F 0 "J12" H 2829 6342 50  0000 L CNN
-F 1 "FAN1" H 2829 6251 50  0000 L CNN
+F 1 "+FAN1-" H 2829 6251 50  0000 L CNN
 F 2 "Felix_Common:PinHeader_1x02_P2.54mm_Vertical_LongPads" H 2750 6350 50  0001 C CNN
 F 3 "~" H 2750 6350 50  0001 C CNN
@@
 P 2750 6700
 F 0 "J13" H 2829 6692 50  0000 L CNN
-F 1 "FAN2" H 2829 6601 50  0000 L CNN
+F 1 "+FAN2-" H 2829 6601 50  0000 L CNN
 F 2 "Felix_Common:PinHeader_1x02_P2.54mm_Vertical_LongPads" H 2750 6700 50  0001 C CNN
 F 3 "~" H 2750 6700 50  0001 C CNN
@@
 P 5850 4550
 F 0 "J20" H 5930 4542 50  0000 L CNN
-F 1 "BED_T" H 5930 4451 50  0000 L CNN
+F 1 "+BT-" H 5930 4451 50  0000 L CNN
 F 2 "Felix_Common:PinHeader_1x02_P2.54mm_Vertical_LongPads" H 5850 4550 50  0001 C CNN
 F 3 "~" H 5850 4550 50  0001 C CNN
@@
 P 7600 4550
 F 0 "J21" H 7679 4542 50  0000 L CNN
-F 1 "NOZZLE_T" H 7679 4451 50  0000 L CNN
+F 1 "+NT-" H 7679 4451 50  0000 L CNN
 F 2 "Felix_Common:PinHeader_1x02_P2.54mm_Vertical_LongPads" H 7600 4550 50  0001 C CNN
 F 3 "~" H 7600 4550 50  0001 C CNN
@@
 P 1700 2050
 F 0 "F1" V 1503 2050 50  0000 C CNN
-F 1 "3A (Rest)" V 1594 2050 50  0000 C CNN
+F 1 "3A REM" V 1594 2050 50  0000 C CNN
 F 2 "Felix_Specials:Fuse_ESKA_380.000" V 1630 2050 50  0001 C CNN
 F 3 "~" H 1700 2050 50  0001 C CNN
@@
 P 1700 1750
 F 0 "F2" V 1503 1750 50  0000 C CNN
-F 1 "10A (Bed)" V 1594 1750 50  0000 C CNN
+F 1 "10A BED" V 1594 1750 50  0000 C CNN
 F 2 "Felix_Specials:Fuse_ESKA_380.000" V 1630 1750 50  0001 C CNN
 F 3 "~" H 1700 1750 50  0001 C CNN
@@
 P 11900 4100
 F 0 "J50" H 11819 3575 50  0000 C CNN
-F 1 "SD_Card" H 11819 3666 50  0000 C CNN
+F 1 "SD    GND" H 11819 3666 50  0000 C CNN
 F 2 "Felix_Common:PinHeader_1x06_P2.54mm_Vertical_LongPads" H 11900 4100 50  0001 C CNN
 F 3 "~" H 11900 4100 50  0001 C CNN
@@
 P 2200 3750
 F 0 "D2" H 2050 3950 50  0000 C CNN
-F 1 "LED_NOZ" H 2050 3850 50  0000 C CNN
+F 1 "NOZ" H 2050 3850 50  0000 C CNN
 F 2 "Felix_Common:LED_D5.0mm" H 2200 3750 50  0001 C CNN
 F 3 "~" H 2200 3750 50  0001 C CNN
@@
 P 1900 5000
 F 0 "D3" H 2000 5250 50  0000 C CNN
-F 1 "LED_BED" H 2000 5150 50  0000 C CNN
+F 1 "BED" H 2000 5150 50  0000 C CNN
 F 2 "Felix_Common:LED_D5.0mm" H 1900 5000 50  0001 C CNN
 F 3 "~" H 1900 5000 50  0001 C CNN
